Commit message: Changes for combined simulation

File: sawyer_description/urdf/sawyer_base.gazebo.xacro (robot description, xacro)
@@ -14,9 +14,9 @@
   <!-- Gazebo-Specific Link Properties -->
 <xacro:if value="$(arg static)">
-  <link name="world"/>
+<!--  <link name="world"/>
   <joint name="fixed" type="fixed">
       <parent link="world"/>
       <child link="base"/>
-  </joint>
+  </joint>-->
 </xacro:if>
 <xacro:if value="$(arg pedestal)">
