Commit message: Sawyer pedestal DAE file updated

File: sawyer_description/urdf/sawyer_base.urdf.xacro (robot description, xacro)
@@ -49,5 +49,5 @@
       <origin rpy="0 0 0" xyz="-0.02 0 -0.29"/>
       <geometry>
-        <cylinder length="0.62" radius="0.18"/>
+        <cylinder length="0.62" radius="0.13"/>
       </geometry>
     </collision>
@@ -58,4 +58,5 @@
     </inertial>
   </link>
+<!--
   <link name="controller_box">
     <collision>
@@ -71,4 +72,5 @@
     <child link="controller_box"/>
   </joint>
+-->
   <link name="pedestal_feet">
     <collision>
